File: BMS-25-Hardware-14S/BMS_25.sch (EAGLE design)
At the start: 218 parts, among them IC1 PBQ79656PAPTQ1, IC2 PBQ79656PAPTQ1, T1 PBHV8115X, 115, T2 PBHV8115X, 115

Commit message: Fixed Ground wiring
Connections:
- removed net CB14-IN: LOW-IN.02, RCB14.1
- removed net CB14-IN-1: HIGH-IN.02, RCB14-1.1
- new net VC14-IN: LOW-IN.01, RVC14.1
- new net VC14-IN-1: HIGH-IN.01, RVC14-1.1
- net BAT: now also LOW-IN.02, RCB14.1; no longer LOW-IN.01, RVC14.1
- net BAT-1: now also HIGH-IN.02, RCB14-1.1; no longer HIGH-IN.01, RVC14-1.1
Changed lines of the file:
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@@
 <net name="BAT" class="0">
 <segment>
-<wire x1="-134.62" y1="-106.68" x2="-129.54" y2="-106.68" width="0.1524" layer="91"/>
-<label x="-134.62" y="-106.68" size="1.778" layer="95" rot="R180"/>
-<pinref part="LOW-IN" gate="G$1" pin="01"/>
-</segment>
-<segment>
-<pinref part="RVC14" gate="G$1" pin="1"/>
-<label x="-66.04" y="-30.48" size="1.778" layer="95"/>
-<wire x1="-53.34" y1="-30.48" x2="-66.04" y2="-30.48" width="0.1524" layer="91"/>
-<wire x1="-53.34" y1="-30.48" x2="-55.88" y2="-30.48" width="0.1524" layer="91"/>
-<wire x1="-55.88" y1="-30.48" x2="-55.88" y2="-20.32" width="0.1524" layer="91"/>
-<junction x="-53.34" y="-30.48"/>
 <pinref part="RBAT" gate="G$1" pin="1"/>
 <wire x1="-55.88" y1="-20.32" x2="55.88" y2="-20.32" width="0.1524" layer="91"/>
@@
 <junction x="55.88" y="-73.66"/>
 <pinref part="RNPN" gate="G$1" pin="1"/>
+<wire x1="-66.04" y1="-27.94" x2="-55.88" y2="-27.94" width="0.1524" layer="91"/>
+<label x="-66.04" y="-27.94" size="1.778" layer="95"/>
+<pinref part="RCB14" gate="G$1" pin="1"/>
+<wire x1="-55.88" y1="-27.94" x2="-35.56" y2="-27.94" width="0.1524" layer="91"/>
+<wire x1="-55.88" y1="-20.32" x2="-55.88" y2="-27.94" width="0.1524" layer="91"/>
+<junction x="-55.88" y="-27.94"/>
+</segment>
+<segment>
+<pinref part="LOW-IN" gate="G$1" pin="02"/>
+<wire x1="-104.14" y1="-106.68" x2="-99.06" y2="-106.68" width="0.1524" layer="91"/>
+<label x="-99.06" y="-106.68" size="1.778" layer="95"/>
 </segment>
 </net>
@@
 <net name="BAT-1" class="0">
 <segment>
-<wire x1="-127" y1="190.5" x2="-121.92" y2="190.5" width="0.1524" layer="91"/>
-<label x="-127" y="190.5" size="1.778" layer="95" rot="R180"/>
-<pinref part="HIGH-IN" gate="G$1" pin="01"/>
-</segment>
-<segment>
-<pinref part="RVC14-1" gate="G$1" pin="1"/>
-<label x="-68.58" y="256.54" size="1.778" layer="95"/>
-<wire x1="-55.88" y1="256.54" x2="-58.42" y2="256.54" width="0.1524" layer="91"/>
-<wire x1="-58.42" y1="256.54" x2="-68.58" y2="256.54" width="0.1524" layer="91"/>
-<wire x1="-58.42" y1="256.54" x2="-58.42" y2="269.24" width="0.1524" layer="91"/>
-<junction x="-58.42" y="256.54"/>
 <pinref part="RBAT-1" gate="G$1" pin="1"/>
 <wire x1="-58.42" y1="269.24" x2="53.34" y2="269.24" width="0.1524" layer="91"/>
@@
 <junction x="53.34" y="215.9"/>
 <pinref part="RNPN-1" gate="G$1" pin="1"/>
+<wire x1="-68.58" y1="259.08" x2="-58.42" y2="259.08" width="0.1524" layer="91"/>
+<label x="-68.58" y="259.08" size="1.778" layer="95"/>
+<pinref part="RCB14-1" gate="G$1" pin="1"/>
+<wire x1="-58.42" y1="259.08" x2="-38.1" y2="259.08" width="0.1524" layer="91"/>
+<wire x1="-58.42" y1="269.24" x2="-58.42" y2="259.08" width="0.1524" layer="91"/>
+<junction x="-58.42" y="259.08"/>
+</segment>
+<segment>
+<pinref part="HIGH-IN" gate="G$1" pin="02"/>
+<wire x1="-96.52" y1="190.5" x2="-91.44" y2="190.5" width="0.1524" layer="91"/>
+<label x="-91.44" y="190.5" size="1.778" layer="95"/>
 </segment>
 </net>
@@
 <wire x1="-104.14" y1="-111.76" x2="-99.06" y2="-111.76" width="0.1524" layer="91"/>
 <label x="-99.06" y="-111.76" size="1.778" layer="95"/>
-</segment>
-</net>
-<net name="CB14-IN" class="0">
-<segment>
-<wire x1="-66.04" y1="-27.94" x2="-35.56" y2="-27.94" width="0.1524" layer="91"/>
-<label x="-66.04" y="-27.94" size="1.778" layer="95"/>
-<pinref part="RCB14" gate="G$1" pin="1"/>
-</segment>
-<segment>
-<pinref part="LOW-IN" gate="G$1" pin="02"/>
-<wire x1="-104.14" y1="-106.68" x2="-99.06" y2="-106.68" width="0.1524" layer="91"/>
-<label x="-99.06" y="-106.68" size="1.778" layer="95"/>
 </segment>
 </net>
@@
 </segment>
 </net>
-<net name="CB14-IN-1" class="0">
-<segment>
-<wire x1="-68.58" y1="259.08" x2="-38.1" y2="259.08" width="0.1524" layer="91"/>
-<label x="-68.58" y="259.08" size="1.778" layer="95"/>
-<pinref part="RCB14-1" gate="G$1" pin="1"/>
-</segment>
-<segment>
-<pinref part="HIGH-IN" gate="G$1" pin="02"/>
-<wire x1="-96.52" y1="190.5" x2="-91.44" y2="190.5" width="0.1524" layer="91"/>
-<label x="-91.44" y="190.5" size="1.778" layer="95"/>
-</segment>
-</net>
 <net name="CB11-IN-1" class="0">
 <segment>
@@
 </segment>
 </net>
+<net name="VC14-IN" class="0">
+<segment>
+<pinref part="RVC14" gate="G$1" pin="1"/>
+<wire x1="-53.34" y1="-30.48" x2="-66.04" y2="-30.48" width="0.1524" layer="91"/>
+<wire x1="-53.34" y1="-30.48" x2="-55.88" y2="-30.48" width="0.1524" layer="91"/>
+<junction x="-53.34" y="-30.48"/>
+<label x="-66.04" y="-30.48" size="1.778" layer="95"/>
+</segment>
+<segment>
+<wire x1="-134.62" y1="-106.68" x2="-129.54" y2="-106.68" width="0.1524" layer="91"/>
+<label x="-134.62" y="-106.68" size="1.778" layer="95" rot="R180"/>
+<pinref part="LOW-IN" gate="G$1" pin="01"/>
+</segment>
+</net>
+<net name="VC14-IN-1" class="0">
+<segment>
+<wire x1="-127" y1="190.5" x2="-121.92" y2="190.5" width="0.1524" layer="91"/>
+<label x="-127" y="190.5" size="1.778" layer="95" rot="R180"/>
+<pinref part="HIGH-IN" gate="G$1" pin="01"/>
+</segment>
+<segment>
+<pinref part="RVC14-1" gate="G$1" pin="1"/>
+<wire x1="-55.88" y1="256.54" x2="-68.58" y2="256.54" width="0.1524" layer="91"/>
+<label x="-68.58" y="256.54" size="1.778" layer="95"/>
+</segment>
+</net>

Commit message: Changed Connectors, pass DRC
Parts:
- HIGH-IN, LOW-IN: value 87606-320LF -> TFM-120-02-L-D; device 87606-320LF:87606-320LF -> TFM-120-02-L-D:TFM-120-02-L-D
Connections:
- removed net CB0-IN: LOW-IN.30, RCB0.1
- removed net CB0-IN-1: HIGH-IN.30, RCB0-1.1
- new net VC0-IN: LOW-IN.11, RVC0.1
- new net VC0-IN-1: HIGH-IN.11, RVC0-1.1
- net BAT: now also LOW-IN.40; no longer LOW-IN.02
- net BAT-1: now also HIGH-IN.40; no longer HIGH-IN.02
- net CB1-IN: now also LOW-IN.14; no longer LOW-IN.28
- net CB1-IN-1: now also HIGH-IN.14; no longer HIGH-IN.28
- net CB10-IN: now also LOW-IN.32; no longer LOW-IN.10
- net CB10-IN-1: now also HIGH-IN.32; no longer HIGH-IN.10
- net CB11-IN: now also LOW-IN.34; no longer LOW-IN.08
- net CB11-IN-1: now also HIGH-IN.34; no longer HIGH-IN.08
- net CB12-IN: now also LOW-IN.36; no longer LOW-IN.06
- net CB12-IN-1: now also HIGH-IN.36; no longer HIGH-IN.06
- net CB13-IN: now also LOW-IN.38; no longer LOW-IN.04
- net CB13-IN-1: now also HIGH-IN.38; no longer HIGH-IN.04
- net CB2-IN: now also LOW-IN.16; no longer LOW-IN.26
- net CB2-IN-1: now also HIGH-IN.16; no longer HIGH-IN.26
- net CB3-IN: now also LOW-IN.18; no longer LOW-IN.24
- net CB3-IN-1: now also HIGH-IN.18; no longer HIGH-IN.24
- net CB4-IN: now also LOW-IN.20; no longer LOW-IN.22
- net CB4-IN-1: now also HIGH-IN.20; no longer HIGH-IN.22
- net CB5-IN: now also LOW-IN.22; no longer LOW-IN.20
- net CB5-IN-1: now also HIGH-IN.22; no longer HIGH-IN.20
- net CB6-IN: now also LOW-IN.24; no longer LOW-IN.18
- net CB6-IN-1: now also HIGH-IN.24; no longer HIGH-IN.18
- net CB7-IN: now also LOW-IN.26; no longer LOW-IN.16
- net CB7-IN-1: now also HIGH-IN.26; no longer HIGH-IN.16
- net CB8-IN: now also LOW-IN.28; no longer LOW-IN.14
- net CB8-IN-1: now also HIGH-IN.28; no longer HIGH-IN.14
- net CB9-IN: now also LOW-IN.30; no longer LOW-IN.12
- net CB9-IN-1: now also HIGH-IN.30; no longer HIGH-IN.12
- net GNDH: now also HIGH-IN.01, HIGH-IN.02, HIGH-IN.12, RCB0-1.1; no longer HIGH-IN.29, HIGH-IN.39, HIGH-IN.40, RVC0-1.1
- net GNDL: now also LOW-IN.01, LOW-IN.02, LOW-IN.12, RCB0.1; no longer LOW-IN.29, LOW-IN.39, LOW-IN.40, RVC0.1
- net TEMP1: now also LOW-IN.09; no longer LOW-IN.31
- net TEMP10: now also HIGH-IN.10; no longer HIGH-IN.32
- net TEMP11: now also HIGH-IN.07; no longer HIGH-IN.33
- net TEMP12: now also HIGH-IN.08; no longer HIGH-IN.34
- net TEMP13: now also HIGH-IN.05; no longer HIGH-IN.35
- net TEMP14: now also HIGH-IN.06; no longer HIGH-IN.36
- net TEMP15: now also HIGH-IN.03; no longer HIGH-IN.37
- net TEMP16: now also HIGH-IN.04; no longer HIGH-IN.38
- net TEMP2: now also LOW-IN.10; no longer LOW-IN.32
- net TEMP3: now also LOW-IN.07; no longer LOW-IN.33
- net TEMP4: now also LOW-IN.08; no longer LOW-IN.34
- net TEMP5: now also LOW-IN.05; no longer LOW-IN.35
- net TEMP6: now also LOW-IN.06; no longer LOW-IN.36
- net TEMP7: now also LOW-IN.03; no longer LOW-IN.37
- net TEMP8: now also LOW-IN.04; no longer LOW-IN.38
- net TEMP9: now also HIGH-IN.09; no longer HIGH-IN.31
- net VC1-IN: now also LOW-IN.13; no longer LOW-IN.27
- net VC1-IN-1: now also HIGH-IN.13; no longer HIGH-IN.27
- net VC10-IN: now also LOW-IN.31; no longer LOW-IN.09
- net VC10-IN-1: now also HIGH-IN.31; no longer HIGH-IN.09
- net VC11-IN: now also LOW-IN.33; no longer LOW-IN.07
- net VC11-IN-1: now also HIGH-IN.33; no longer HIGH-IN.07
- net VC12-IN: now also LOW-IN.35; no longer LOW-IN.05
- net VC12-IN-1: now also HIGH-IN.35; no longer HIGH-IN.05
- net VC13-IN: now also LOW-IN.37; no longer LOW-IN.03
- net VC13-IN-1: now also HIGH-IN.37; no longer HIGH-IN.03
- net VC14-IN: now also LOW-IN.39; no longer LOW-IN.01
- net VC14-IN-1: now also HIGH-IN.39; no longer HIGH-IN.01
- net VC2-IN: now also LOW-IN.15; no longer LOW-IN.25
- net VC2-IN-1: now also HIGH-IN.15; no longer HIGH-IN.25
- net VC3-IN: now also LOW-IN.17; no longer LOW-IN.23
- net VC3-IN-1: now also HIGH-IN.17; no longer HIGH-IN.23
- net VC4-IN: now also LOW-IN.19; no longer LOW-IN.21
- net VC4-IN-1: now also HIGH-IN.19; no longer HIGH-IN.21
- net VC5-IN: now also LOW-IN.21; no longer LOW-IN.19
- net VC5-IN-1: now also HIGH-IN.21; no longer HIGH-IN.19
- net VC6-IN: now also LOW-IN.23; no longer LOW-IN.17
- net VC6-IN-1: now also HIGH-IN.23; no longer HIGH-IN.17
- net VC7-IN: now also LOW-IN.25; no longer LOW-IN.15
- net VC7-IN-1: now also HIGH-IN.25; no longer HIGH-IN.15
- net VC8-IN: now also LOW-IN.27; no longer LOW-IN.13
- net VC8-IN-1: now also HIGH-IN.27; no longer HIGH-IN.13
- net VC9-IN: now also LOW-IN.29; no longer LOW-IN.11
- net VC9-IN-1: now also HIGH-IN.29; no longer HIGH-IN.11
