File: BMS_25_Daughter/BMS_25.brd (EAGLE design)
At the start: 140.3 x 51.7 mm, 178 parts, among them IC1 PBQ79656PAPTQ1, IC2 PBQ79656PAPTQ1, T1 PBHV8115X, 115, T2 PBHV8115X, 115

Commit message: Updated Change to daughteboard 14s for final manufacturing
Parts:
- removed CCOMHN, CCOMHP, CCOMLN, CCOMLP, CISOL, CISOL1: 2.2nF, NFR23_v1.3:C0603
- added C1, C2, C3, C4, C5, C6: C1206C105K5RACTU, C1206C105K5RACTU:CAPC3216X120N
- added TP1, TP2, TP3, TP4: 5002, 5002:KEYSTONE_5002
- moved RCOMH 0.37 mm to (69.5, 31.4)
- moved RCOMH1 0.30 mm to (69.5, 25.1)
- moved RCOML1-1 0.10 mm to (77.3, 24.9)
Connections:
- net GNDH: now also TP4.TP
- net GNDL: now also TP2.TP
- net ISO_COMN: now also C4.2; no longer CISOL1.1
- net ISO_COMP: now also C3.2; no longer CISOL.1
- net N$101: now also C2.2; no longer CCOMHN.1
- net N$103: now also C5.1; no longer CCOMLN.1
- net N$104: now also C6.1; no longer CCOMLP.1
- net N$46: now also C3.1; no longer CISOL.2
- net N$47: now also C4.1; no longer CISOL1.2
- net N$50: now also C5.2; no longer CCOMLN.2
- net N$51: now also C6.2; no longer CCOMLP.2
- net N$97: now also C1.1; no longer CCOMHP.2
- net N$98: now also C2.1; no longer CCOMHN.2
- net N$99: now also C1.2; no longer CCOMHP.1
- net TP: now also TP3.TP
- net TP-1: now also TP1.TP
Routing:
- net BAT-1: track 69.0 -> 72.6 mm
- net TP-1: track 11.6 -> 15.1 mm
- net GNDL: track 50.3 -> 53.8 mm
- net GNDH: track 42.8 -> 45.9 mm
- net TP: track 24.2 -> 27.2 mm
- net N$101: track 4.78 -> 3.71 mm
- net N$104: track 4.27 -> 3.27 mm
- net N$99: track 4.95 -> 4.12 mm
- net N$51: track 6.76 -> 6.17 mm
- net ISO_COMP: track 2.11 -> 1.58 mm
